File: AirPurifier/AirPurifier.kicad_sch (KiCad schematic)
At the start: 0 parts

Commit message: update
Other:
- added sheet OpticSensor (./AP_OpticSensor/OpticSensor.kicad_sch)
- added sheet PIRSensor (./AP_PIRSensor/PIRSensor.kicad_sch)
- sheet MCU: file .\AP_MCU\MCU.kicad_sch -> ./AP_MCU/MCU.kicad_sch
- sheet MotorControl: file MotorControl.kicad_sch -> ./AP_MotorControl/AP_MotroControl.kicad_sch
Changed lines of the file:
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@@
 (kicad_sch (version 20211123) (generator eeschema)
   (paper "A4")
-  (sheet (at 124.46 24.13) (size 39.37 26.67) (fields_autoplaced)
+  (sheet (at 121.92 35.56) (size 30.48 25.4) (fields_autoplaced)
     (stroke (width 0.1524) (type solid) (color 0 0 0 0))
     (fill (color 0 0 0 0.0000))
-    (property "Sheet name" "MCU" (id 0) (at 124.46 23.4184 0)
+    (property "Sheet name" "MCU" (id 0) (at 121.92 34.8484 0)
       (effects (font (size 1.27 1.27)) (justify left bottom))
     )
-    (property "Sheet file" ".\\AP_MCU\\MCU.kicad_sch" (id 1) (at 124.46 51.3846 0)
+    (property "Sheet file" "./AP_MCU/MCU.kicad_sch" (id 1) (at 121.92 61.5446 0)
       (effects (font (size 1.27 1.27)) (justify left top))
     )
   )
-  (sheet (at 168.91 78.74) (size 68.58 33.02) (fields_autoplaced)
+  (sheet (at 160.02 35.56) (size 30.48 25.4) (fields_autoplaced)
     (stroke (width 0.1524) (type solid) (color 0 0 0 0))
     (fill (color 0 0 0 0.0000))
-    (property "Sheet name" "MotorControl" (id 0) (at 168.91 78.0284 0)
+    (property "Sheet name" "MotorControl" (id 0) (at 160.02 34.8484 0)
       (effects (font (size 1.27 1.27)) (justify left bottom))
     )
-    (property "Sheet file" "MotorControl.kicad_sch" (id 1) (at 168.91 112.3446 0)
+    (property "Sheet file" "./AP_MotorControl/AP_MotroControl.kicad_sch" (id 1) (at 160.02 61.5446 0)
+      (effects (font (size 1.27 1.27)) (justify left top))
+    )
+  )
+  (sheet (at 213.36 35.56) (size 30.48 25.4) (fields_autoplaced)
+    (stroke (width 0.1524) (type solid) (color 0 0 0 0))
+    (fill (color 0 0 0 0.0000))
+    (property "Sheet name" "OpticSensor" (id 0) (at 213.36 34.8484 0)
+      (effects (font (size 1.27 1.27)) (justify left bottom))
+    )
+    (property "Sheet file" "./AP_OpticSensor/OpticSensor.kicad_sch" (id 1) (at 213.36 61.5446 0)
+      (effects (font (size 1.27 1.27)) (justify left top))
+    )
+  )
+  (sheet (at 213.36 68.58) (size 30.48 25.4) (fields_autoplaced)
+    (stroke (width 0.1524) (type solid) (color 0 0 0 0))
+    (fill (color 0 0 0 0.0000))
+    (property "Sheet name" "PIRSensor" (id 0) (at 213.36 67.8684 0)
+      (effects (font (size 1.27 1.27)) (justify left bottom))
+    )
+    (property "Sheet file" "./AP_PIRSensor/PIRSensor.kicad_sch" (id 1) (at 213.36 94.5646 0)
       (effects (font (size 1.27 1.27)) (justify left top))
     )
@@
   (sheet_instances
     (path "/" (page "1"))
-    (path "/503dbd88-3e6b-48cc-a2ea-a6e28b52a1f7" (page "2"))
     (path "/088f77ba-fca9-42b3-876e-a6937267f957" (page "3"))
+    (path "/1cca5857-ed00-42ca-b889-3671b0d9e1b3" (page "3"))
+    (path "/2af1c65a-1e67-405a-9e99-0802dde719e5" (page "4"))
+    (path "/33f45502-c1c8-4769-a0a3-a77f7eed1f55" (page "5"))
   )
   (symbol_instances
